File: hardware/motherboard_rev_3/motherboard_rev_3.kicad_sch (KiCad schematic)
At the start: 42 parts, among them J1 Conn_ST_STDC14, J2 USB_C_Receptacle_USB2.0, J3 EH_S8B-EH, U1 GPS module, U10 SCD41-D-R2, U2 ICM-42688, U3 STM32F412CGU6, U4 BMP390, U5 BME280, U6 nRF24L01, U7 nRF24L01, U8 USBLC6-2SC6, U9 BNO055, Y1 20M

Commit message: Added schematic for future integrated nRF24 modules
Other:
- added sheet nRF24 Comms (nrf24.kicad_sch)
Changed lines of the file:
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@@
+	)
+	(sheet
+		(at 190.5 180.34)
+		(size 67.31 33.02)
+		(exclude_from_sim no)
+		(in_bom yes)
+		(on_board yes)
+		(dnp no)
+		(fields_autoplaced yes)
+		(stroke
+			(width 0.1524)
+			(type solid)
+		)
+		(fill
+			(color 0 0 0 0.0000)
+		)
+		(property "Sheetname" "nRF24 Comms"
+			(at 190.5 179.6284 0)
+			(effects
+				(font
+					(size 1.27 1.27)
+				)
+				(justify left bottom)
+			)
+		)
+		(property "Sheetfile" "nrf24.kicad_sch"
+			(at 190.5 213.9446 0)
+			(effects
+				(font
+					(size 1.27 1.27)
+				)
+				(justify left top)
+			)
+		)
+		(instances
+			(project "motherboard_rev_3"
+				(path "/39c7ec0f-0a05-4172-b48a-dcc9b63f77ff"
+					(page "4")
+				)
+			)
+		)
 	)
 	(sheet

Commit message: Motherboard rev 3.1 as ordered
Parts:
- C1, C10, C12, C13, C3, C5, C6, C7, C8, C9: LCSC C5448875 -> C301928
- J2: value USB_C_Receptacle_USB2.0 -> USB4105-GF-A-120; footprint Connector_USB:USB_C_Receptacle_HRO_TYPE-C-31-M-12 -> Connector_USB:USB_C_Receptacle_GCT_USB4105-xx-A_16P_TopMnt_Horizontal; LCSC C165948 -> C5184243
Other:
- removed sheet nRF24 Comms
Changed lines of the file:
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@@
 	(title_block
 		(title "Falcon Motherboard")
-		(date "2025-08-20")
-		(rev "3.0")
+		(date "2025-08-23")
+		(rev "3.1")
 		(company "HPVDT")
 		(comment 1 "Revised connections for programming pins")
@@
 			)
 		)
-		(property "Value" "USB_C_Receptacle_USB2.0"
+		(property "Value" "USB4105-GF-A-120"
 			(at 386.08 44.4499 0)
 			(effects
@@
 			)
 		)
-		(property "Footprint" "Connector_USB:USB_C_Receptacle_HRO_TYPE-C-31-M-12"
+		(property "Footprint" "Connector_USB:USB_C_Receptacle_GCT_USB4105-xx-A_16P_TopMnt_Horizontal"
 			(at 370.84 43.18 0)
 			(effects
@@
 			)
 		)
-		(property "LCSC" "C165948"
+		(property "LCSC" "C5184243"
 			(at 374.65 43.18 0)
 			(effects
@@
 			)
 		)
-		(property "LCSC" "C5448875"
+		(property "LCSC" "C301928"
 			(at 127 231.14 0)
 			(effects
@@
 			)
 		)
-		(property "LCSC" "C5448875"
+		(property "LCSC" "C301928"
 			(at 171.45 39.37 0)
 			(effects
@@
 			)
 		)
-		(property "LCSC" "C5448875"
+		(property "LCSC" "C301928"
 			(at 133.35 231.14 0)
 			(effects
@@
 			)
 		)
-		(property "LCSC" "C5448875"
+		(property "LCSC" "C301928"
 			(at 147.32 39.37 0)
 			(effects
@@
 			)
 		)
-		(property "LCSC" "C5448875"
+		(property "LCSC" "C301928"
 			(at 158.75 39.37 0)
 			(effects
@@
 			)
 		)
-		(property "LCSC" "C5448875"
+		(property "LCSC" "C301928"
 			(at 44.45 242.57 0)
 			(effects
@@
 			)
 		)
-		(property "LCSC" "C5448875"
+		(property "LCSC" "C301928"
 			(at 99.06 173.99 0)
 			(effects
@@
 			)
 		)
-		(property "LCSC" "C5448875"
+		(property "LCSC" "C301928"
 			(at 312.42 184.15 0)
 			(effects
@@
 			)
 		)
-		(property "LCSC" "C5448875"
+		(property "LCSC" "C301928"
 			(at 92.71 173.99 0)
 			(effects
@@
 			)
 		)
-		(property "LCSC" "C5448875"
+		(property "LCSC" "C301928"
 			(at 299.72 184.15 0)
 			(effects
@@
 				)
 			)
-		)
-	)
-	(sheet
-		(at 190.5 180.34)
-		(size 67.31 33.02)
-		(exclude_from_sim no)
-		(in_bom yes)
-		(on_board yes)
-		(dnp no)
-		(fields_autoplaced yes)
-		(stroke
-			(width 0.1524)
-			(type solid)
-		)
-		(fill
-			(color 0 0 0 0.0000)
-		)
-		(property "Sheetname" "nRF24 Comms"
-			(at 190.5 179.6284 0)
-			(effects
-				(font
-					(size 1.27 1.27)
-				)
-				(justify left bottom)
-			)
-		)
-		(property "Sheetfile" "nrf24.kicad_sch"
-			(at 190.5 213.9446 0)
-			(effects
-				(font
-					(size 1.27 1.27)
-				)
-				(justify left top)
-			)
-		)
-		(instances
-			(project "motherboard_rev_3"
-				(path "/39c7ec0f-0a05-4172-b48a-dcc9b63f77ff"
-					(page "4")
-				)
-			)
